File: KiCad/Ingressi/Ingressi.kicad_pcb (KiCad board)
At the start: 2 copper layers, 100 x 65 mm, 4 parts, among them J1 SpeakON_NL4, J2 SpeakON_NL4, J3 Phoenix MKDS, J4 JST_S4P-VH

Commit message: updated PCB
Parts:
- added G***: LOGO, Stakx logo:stakx_small_fp, B.Cu at (75.0, 63.0)
- moved J4 1.87 mm to (88.7, 75.4)
- moved J3 0.95 mm to (52.7, 80.7)
Routing:
- added copper zone on F.Cu, net Net-(J1-Pad1+)
- added copper zone on B.Cu, net Net-(J1-Pad1-)
- added copper zone on F.Cu, net Net-(J1-Pad2+)
- added copper zone on B.Cu, net Net-(J1-Pad2-)
Other:
- board text added: "1+"
- board text added: "1-"
- board text added: "2+"
- board text added: "2-"
